Commit message: UPDATE: 2 Finger Gripper

File: UR5+gripper/ur5_gripper.urdf (robot description, URDF)
Before this commit: robot ur5, 52 links, 51 joints
Joints:
- joint shoulder_lift_joint: limit lower=-3.14159265 upper=-1.0 effort=150.0 velocity=3.15 -> lower=-3.14159265 upper=-0.9 effort=150.0 velocity=3.15
